File: BLDC__MD_Mounter/BLDC__MD_Mounter.kicad_pcb (KiCad board)
At the start: 2 copper layers, 64 x 60 mm, 18 parts, among them J1 Conn_02x07_Odd_Even, J10 Conn_02x07_Odd_Even, J11 Conn_01x08_Female, J12 Conn_02x07_Odd_Even, J13 Conn_02x07_Odd_Even, J14 Conn_01x08_Female, J2 Conn_02x07_Odd_Even, J3 Conn_02x10_Odd_Even, J4 Conn_01x08_Female, J5 Conn_01x02_Male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

Commit message: #fix reverse pin sockets bottom and sig port pin socket.
Parts:
- moved J3 23.0 mm to (156.3, 88.3), turned to 180 degrees
- moved J11 17.8 mm to (131.2, 105.7), turned to 180 degrees
- moved J14 17.8 mm to (141.8, 105.7), turned to 180 degrees
- moved J4 17.8 mm to (110.0, 105.7), turned to 180 degrees
- moved J8 17.8 mm to (120.6, 105.7), turned to 180 degrees
Connections:
- J3 pad 1: +3V3 -> Net-(J3-Pad1)
- J3 pad 10: /PWM_3 -> /FR_2
- J3 pad 11: /FG_1 -> /RD_4
- J3 pad 12: /RD_3 -> /FG_2
- J3 pad 13: /RD_2 -> /FG_3
- J3 pad 14: /FG_4 -> /RD_1
- J3 pad 15: /PWM_2 -> /FR_3
- J3 pad 16: /FR_4 -> /PWM_1
- J3 pad 17: /FR_2 -> /PWM_3
- J3 pad 18: /PWM_4 -> /FR_1
- J3 pad 19: /FG_2 -> /RD_3
- J3 pad 2: Net-(J3-Pad2) -> +5V
- J3 pad 20: /RD_4 -> /FG_1
- J3 pad 3: +5V -> GND
- J3 pad 4: GND -> +3V3
- J3 pad 5: /RD_1 -> /FG_4
- J3 pad 6: /FG_3 -> /RD_2
- J3 pad 7: /PWM_1 -> /FR_4
- J3 pad 8: /FR_3 -> /PWM_2
- J3 pad 9: /FR_1 -> /PWM_4
Routing:
- net /FG_2: track 72.6 -> 37.6 mm
- net /FG_1: track 78.2 -> 46.6 mm
- net /FR_2: track 68.6 -> 40.5 mm
- net /FR_1: track 74.6 -> 49.2 mm
- net /PWM_2: track 65.0 -> 44.0 mm
- net VCC: track 78.4 -> 58.3 mm
- net /RD_3: track 48.4 -> 68.4 mm
- net /RD_4: track 21.3 -> 41.1 mm
- net /PWM_1: track 71.1 -> 52.4 mm
- net /PWM_3: track 50.4 -> 66.4 mm
- net /RD_2: track 61.4 -> 47.0 mm
- net /PWM_4: track 24.5 -> 38.6 mm
- net /RD_1: track 67.5 -> 54.4 mm
- net /FR_3: track 53.2 -> 64.3 mm
- net /FR_4: track 26.5 -> 36.8 mm
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